File: ergogen/output/pcbs/simple34_v2.kicad_pcb (KiCad board)
At the start: 2 copper layers, 122.2 x 90.8 mm, 42 parts

Commit message: OH MY, ARCS EXISTS
Parts:
- removed RST1: , ceoloide:reset_switch_tht_top
- added SW1: , local:reset_smd, F.Cu at (137.9, 87.2)
- moved H4 32.0 mm to (121.8, 96.0), turned to -17.5 degrees
- moved H1 18.6 mm to (45.4, 53.5)
- moved H2 16.0 mm to (110.4, 34.7)
- moved H3 14.6 mm to (58.4, 101.8)
- moved D17 11.4 mm to (131.7, 100.5)
- moved D16 11.4 mm to (111.1, 94.0)
- moved JST1 10.6 mm to (128.9, 86.2), turned to 90 degrees
- moved D6 8.50 mm to (58.1, 40.4)
- moved D4 8.50 mm to (61.1, 74.3)
- moved D5 8.50 mm to (59.6, 57.4)
- moved D14 8.50 mm to (116.4, 58.5)
- moved D10 8.50 mm to (98.4, 72.7)
- moved D12 8.50 mm to (98.4, 38.7)
- moved D13 8.50 mm to (116.4, 75.5)
- moved D15 8.50 mm to (116.4, 41.5)
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Connections:
- JST1 pad 1: BAT_P -> GND
- JST1 pad 2: GND -> BAT_P
- S1 pad 1: pinky_bottom -> C0
- S10 pad 1: index_bottom -> C3
- S11 pad 1: index_home -> C3
- S12 pad 1: index_top -> C3
- S13 pad 1: inner_bottom -> C4
- S14 pad 1: inner_home -> C4
- S15 pad 1: inner_top -> C4
- S16 pad 1: first_only -> C4
- S17 pad 1: second_only -> C5
- S2 pad 1: pinky_home -> C0
- S3 pad 1: pinky_top -> C0
- S4 pad 1: ring_bottom -> C1
- S5 pad 1: ring_home -> C1
- S6 pad 1: ring_top -> C1
- S7 pad 1: middle_bottom -> C2
- S8 pad 1: middle_home -> C2
- S9 pad 1: middle_top -> C2
Routing:
- net C4: track 177.6 -> 122.3 mm, vias 3 -> 6
- net C0: track 229.2 -> 184.3 mm, vias 1 -> 3
- net C3: track 159.5 -> 116.6 mm, vias 1 -> 5
- net C2: track 182.7 -> 140.1 mm, vias 1 -> 5
- net C1: track 200.9 -> 160.0 mm, vias 1 -> 5
- net RAW: track 88.5 -> 47.8 mm, vias 5 -> 2
- net C5: track 83.2 -> 56.0 mm, vias 0 -> 2
- net RST: track 62.1 -> 35.3 mm, vias 2 -> 1
- net R1: track 148.4 -> 134.1 mm, vias 5 -> 0
- net R0: track 165.5 -> 151.7 mm, vias 7 -> 1
- net R3: track 65.5 -> 52.6 mm
- net BAT_P: track 7.03 -> 18.1 mm
- net GND: track 91.0 -> 81.0 mm, vias 4 -> 3
- net R2: track 129.5 -> 120.8 mm, vias 5 -> 1
- net JST1_2: track 3.60 -> 0.00 mm
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- added copper zone on B.Cu, net GND
- added copper zone on F.Cu, net GND
- removed copper zone on B.Cu, net (none)
- removed copper zone on F.Cu, net (none)
Other:
- board size 122.2 x 90.8 mm -> 120 x 89.4 mm
- board text removed: "- +"

Commit message: case fillet
Parts:
- removed H3, H4: , ceoloide:mounting_hole_plated
- added TP1: Tenting Puck, no hole, TentingPuck_NoHole, B.Cu at (93.4, 61.6)
- moved H1 99.5 mm to (134.2, 98.6), turned to -25 degrees
- moved H2 76.4 mm to (144.1, 103.3), turned to -25 degrees
- moved D15 16.4 mm to (119.9, 57.5), turned to 360 degrees
- moved S7 9.83 mm to (83.9, 80.9)
- moved D8 9.83 mm to (83.9, 59.2)
- moved D9 9.83 mm to (83.9, 42.2)
- moved S8 9.83 mm to (83.9, 63.9)
- moved S9 9.83 mm to (83.9, 46.9)
- moved D7 9.83 mm to (83.9, 76.2)
- moved D6 8.52 mm to (62.4, 47.8), turned to 184 degrees
- moved D10 8.52 mm to (101.9, 80.4)
- moved S11 8.52 mm to (101.9, 68.1)
- moved S12 8.52 mm to (101.9, 51.1)
- moved D11 8.52 mm to (101.9, 63.4)
- moved D12 8.52 mm to (101.9, 46.4)
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Routing:
- net (no net): track 0.00 -> 337.7 mm
- net C0: track 184.3 -> 24.8 mm
- net R0: track 151.7 -> 0.00 mm, vias 1 -> 0
- net C1: track 160.0 -> 24.8 mm, vias 5 -> 3
- net R1: track 134.1 -> 0.00 mm
- net R2: track 120.8 -> 0.00 mm, vias 1 -> 0
- net C2: track 140.1 -> 24.8 mm, vias 5 -> 3
- net C3: track 116.6 -> 24.8 mm, vias 5 -> 3
- net C4: track 122.3 -> 33.1 mm, vias 6 -> 4
- net GND: track 81.0 -> 0.00 mm, vias 3 -> 0
- net R3: track 52.6 -> 0.00 mm, vias 2 -> 0
- net RAW: track 47.8 -> 0.00 mm, vias 2 -> 0
- net C5: track 56.0 -> 8.27 mm, vias 2 -> 1
- net RST: track 35.3 -> 0.00 mm, vias 1 -> 0
- net BAT_P: track 18.1 -> 0.00 mm, vias 1 -> 0
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- removed copper zone on B.Cu, net GND
- removed copper zone on F.Cu, net GND
Other:
- board size 120 x 89.4 mm -> 116.6 x 89.6 mm

Commit message: huge change
Routing:
- net (no net): track 337.7 -> 0.00 mm
- net C0: track 24.8 -> 180.7 mm
- net C1: track 24.8 -> 165.4 mm, vias 3 -> 4
- net R0: track 0.00 -> 132.8 mm
- net R1: track 0.00 -> 123.8 mm
- net C2: track 24.8 -> 142.7 mm, vias 3 -> 4
- net R2: track 0.00 -> 110.3 mm
- net C4: track 33.1 -> 142.5 mm, vias 4 -> 5
- net C3: track 24.8 -> 120.9 mm, vias 3 -> 4
- net GND: track 0.00 -> 70.4 mm, vias 0 -> 2
- net R3: track 0.00 -> 51.5 mm, vias 0 -> 1
- net C5: track 8.27 -> 57.1 mm, vias 1 -> 2
- net RAW: track 0.00 -> 47.8 mm, vias 0 -> 2
- net RST: track 0.00 -> 38.0 mm, vias 0 -> 2
- net BAT_P: track 0.00 -> 18.1 mm, vias 0 -> 1
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- added copper zone on B.Cu, net GND
- added copper zone on F.Cu, net GND
Other:
- outline, holes or cut-outs redrawn

Commit message: LARGE UPDATE
Parts:
- removed H1, H2: , ceoloide:mounting_hole_plated
- removed JST1: , ceoloide:battery_connector_jst_ph_2
- added BAT1: , terence:battery_socket_tht, F.Cu at (139.4, 63.3)
- added LED1: , terence:led_5mm_tht, F.Cu at (144.9, 97.8)
- added LED2: , terence:led_5mm_tht, F.Cu at (139.4, 97.8)
- added LED3: , terence:led_5mm_tht, F.Cu at (133.9, 97.8)
- added R1: , terence:resistor_1206, F.Cu at (142.4, 103.8)
- added R2: , terence:resistor_1206, F.Cu at (139.4, 103.8)
- added R3: , terence:resistor_1206, F.Cu at (136.4, 103.8)
- moved PWR1 33.3 mm to (139.4, 63.3), turned to 90 degrees
- moved SW1 11.7 mm to (128.4, 97.8), turned to 90 degrees
- moved D15 9.40 mm to (119.9, 48.1), turned to 180 degrees
- moved MCU1 4.00 mm to (139.4, 78.3)
- turned S15 to 180 degrees
Connections:
- MCU1 pad 117: P5 -> led_3
- MCU1 pad 118: P4 -> led_2
- MCU1 pad 119: P3 -> led_1
- S1 pad 1: C0 -> pinky_bottom
- S1 pad 2: pinky_bottom -> C0
- S10 pad 1: C3 -> index_bottom
- S10 pad 2: index_bottom -> C3
- S11 pad 1: C3 -> index_home
- S11 pad 2: index_home -> C3
- S12 pad 1: C3 -> index_top
- S12 pad 2: index_top -> C3
- S13 pad 1: C4 -> inner_bottom
- S13 pad 2: inner_bottom -> C4
- S14 pad 1: C4 -> inner_home
- S14 pad 2: inner_home -> C4
- S15 pad 1: C4 -> inner_top
- S15 pad 2: inner_top -> C4
- S16 pad 1: C4 -> first_only
- S16 pad 2: first_only -> C4
- S17 pad 1: C5 -> second_only
- S17 pad 2: second_only -> C5
- S2 pad 1: C0 -> pinky_home
- S2 pad 2: pinky_home -> C0
- S3 pad 1: C0 -> pinky_top
- S3 pad 2: pinky_top -> C0
- S4 pad 1: C1 -> ring_bottom
- S4 pad 2: ring_bottom -> C1
- S5 pad 1: C1 -> ring_home
- S5 pad 2: ring_home -> C1
- S6 pad 1: C1 -> ring_top
- S6 pad 2: ring_top -> C1
- S7 pad 1: C2 -> middle_bottom
- S7 pad 2: middle_bottom -> C2
- S8 pad 1: C2 -> middle_home
- S8 pad 2: middle_home -> C2
- S9 pad 1: C2 -> middle_top
- S9 pad 2: middle_top -> C2
Routing:
- net C4: track 142.5 -> 96.8 mm, vias 5 -> 2
- net led_1: track 0.00 -> 34.6 mm
- net RAW: track 47.8 -> 15.6 mm
- net led_2: track 0.00 -> 28.7 mm
- net C3: track 120.9 -> 93.2 mm, vias 4 -> 1
- net C2: track 142.7 -> 115.2 mm, vias 4 -> 1
- net C1: track 165.4 -> 138.0 mm, vias 4 -> 1
- net led_3: track 0.00 -> 25.2 mm
- net C0: track 180.7 -> 161.5 mm, vias 3 -> 0
- net GND: track 70.4 -> 55.0 mm
- net R0: track 132.8 -> 146.2 mm
- net BAT_P: track 18.1 -> 5.91 mm
- net r3: track 0.00 -> 12.1 mm
- net r2: track 0.00 -> 10.1 mm
- net r1: track 0.00 -> 10.0 mm
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Other:
- board size 116.6 x 89.6 mm -> 114.6 x 86.5 mm

Commit message: lil change
Parts:
- moved LED3 2.06 mm to (131.9, 98.3), turned to 180 degrees
- moved LED2 1.58 mm to (137.9, 98.3), turned to 180 degrees
- moved R1 1.58 mm to (140.9, 103.3)
- moved R2 1.58 mm to (137.9, 103.3)
- moved R3 1.58 mm to (134.9, 103.3)
- moved SW1 1.58 mm to (126.9, 98.3)
- moved BAT1 1.50 mm to (137.9, 63.3)
- moved MCU1 1.50 mm to (137.9, 78.3)
- moved PWR1 1.50 mm to (137.9, 63.3)
- moved LED1 1.12 mm to (143.9, 98.3), turned to 180 degrees
Routing:
- net R2: track 115.4 -> 111.4 mm
- net r3: track 12.1 -> 8.43 mm
- net R3: track 50.7 -> 47.4 mm
- net C0: track 161.5 -> 158.9 mm
- net R1: track 129.0 -> 126.9 mm
- net R0: track 146.2 -> 144.2 mm
- net r2: track 10.1 -> 8.05 mm
- net led_3: track 25.2 -> 27.0 mm
- net C2: track 115.2 -> 113.8 mm
- net r1: track 10.0 -> 11.4 mm
- net led_1: track 34.6 -> 33.2 mm
- net C1: track 138.0 -> 136.7 mm
- net led_2: track 28.7 -> 28.2 mm
Other:
- board size 114.6 x 86.5 mm -> 113.1 x 86.5 mm

Commit message: another change
Routing:
- net r1: track 11.4 -> 6.70 mm, vias 0 -> 1
- net r3: track 8.43 -> 4.23 mm, vias 0 -> 1
- net r2: track 8.05 -> 4.03 mm, vias 0 -> 1
- net C4: track 96.7 -> 93.6 mm
- net C3: track 93.3 -> 91.2 mm
- net R2: track 111.4 -> 113.1 mm
- net C5: track 50.0 -> 48.4 mm
- net R1: track 126.9 -> 128.5 mm
- net R0: track 144.2 -> 143.6 mm
- net C1: track 136.7 -> 136.2 mm
- net GND: track 54.6 -> 54.9 mm, vias 2 -> 0
